File: XT Prototype Board.kicad_pcb (KiCad board)
At the start: 2 copper layers, 101.6 x 101.6 mm, 5 parts, among them J1 Bus_ISA_8bit, J2 Breakout

Commit message: Add files via upload
Parts:
- removed LOGO1, LOGO2: LOGO, Custom:Monotech Logo 12.7mm
- added G***: LOGO, Custom:LOGO, F.Cu at (60.3, 125.1)
- added LOGOBACK: LOGO, Custom:LOGO, B.Cu at (60.3, 125.1)
Connections:
- net ~DACK0 renamed ~{DACK0}
- net ~DACK1 renamed ~{DACK1}
- net ~DACK2 renamed ~{DACK2}
- net ~DACK3 renamed ~{DACK3}
- net ~IOR renamed ~{IOR}
- net ~IOW renamed ~{IOW}
- net ~MEMR renamed ~{MEMR}
- net ~MEMW renamed ~{MEMW}
Other:
- net class Default removed
- rule pad_to_mask_clearance: 0.051 -> 0
- board text added: "The Wizard"
- board text added: "~{DACK0}"
- board text added: "~{DACK1}"
- board text added: "~{DACK2}"
- board text added: "~{DACK3}"
- board text added: "~{IOR}"
- board text added: "~{IOW}"
- board text added: "~{MEMR}"
- board text added: "~{MEMW}"
- board text removed: "Monotech PCs"
- board text removed: "~DACK0"
- board text removed: "~DACK1"
- board text removed: "~DACK2"
- board text removed: "~DACK3"
- board text removed: "~IOR"
- board text removed: "~IOW"
- board text removed: "~MEMR"
- board text removed: "~MEMW"
